Commit message: Avances

File: ExamenParcial2/ros2_ws/src/scara_description/urdf/scara.urdf (robot description, URDF)
Before this commit: robot scara, 5 links, 4 joints
Links:
- removed link link1
- removed link link2
- removed link link3
- removed link link4
- added link link_1, mass 1; collision box size=0.5 0.05 0.05; visual box size=0.5 0.05 0.05
- added link link_2, mass 1; collision box size=0.5 0.05 0.05; visual box size=0.5 0.05 0.05
- added link link_3, mass 1; collision box size=0.3 0.05 0.05; visual box size=0.3 0.05 0.05
- link base_link: mass 12.72 -> 1; geometry collision box size=0.1 0.15 0.2; visual box size=0.1 0.15 0.2
Joints:
- removed joint scara_joint1
- removed joint scara_joint2
- removed joint scara_joint3
- removed joint scara_joint4
- added joint link_1_joint: type revolute, parent base_link, child link_1, origin xyz=0 0 0.225 rpy=0 0 0, axis 0 0 1, limit lower=-3.14159 upper=3.14159 effort=1000.0 velocity=50.0
- added joint link_2_joint: type revolute, parent link_1, child link_2, origin xyz=0.45 0 0.05 rpy=0 0 0, axis 0 0 1, limit lower=-3.14159 upper=3.14159 effort=1000.0 velocity=50.0
- added joint link_3_joint: type revolute, parent link_2, child link_3, origin xyz=0.45 0 -0.05 rpy=0 0 0, axis 0 0 1, limit lower=-3.14159 upper=3.14159 effort=1000.0 velocity=50.0
